File: schematics/clock/clock.kicad_sch (KiCad schematic)
At the start: 26 parts, among them SW1 SW_DIP_x12, U1 4060, U10 74HC00, U11 28C64, U2 4060, U3 74HC163, U4 74HC163, U5 74HC30, U6 74HC163, U7 74HC163, U8 74HC163, U9 74HC30, Y1 32.768khz

Commit message: finished first revision of schematic
Parts:
- added U12: CC5641AS, Display_7Segment:CA56-12SRWA, symbol Display_Character:CC56-12SRWA
- added U13: 74HC109, symbol My_Symbols:74HC109
- added U14: 74HC139, symbol My_Symbols:74HC139
Connections:
- net +5V: now also U11.27 (~{WE}), U11.28 (VCC), U13.1 (~{R}), U13.11 (~{S}), U13.14 (J), U13.15 (~{R}), U13.2 (J), U13.5 (~{S})
- net GND: now also U11.14 (GND), U11.20 (~{CE}), U11.22 (~{OE}), U13.13 (~{K}), U13.3 (~{K}), U14.1 (E)
- net T0: no longer U11.21 (A10), U11.24 (A9), U11.25 (A8), U11.3 (A7), U11.4 (A6), U11.5 (A5), U11.6 (A4), U11.7 (A3), U11.8 (A2)
- net T10: now also U11.21 (A10)
- net T2: now also U11.8 (A2)
- net T3: now also U11.7 (A3)
- net T4: now also U11.6 (A4)
- net T5: now also U11.5 (A5)
- net T6: now also U11.4 (A6)
- net T7: now also U11.3 (A7)
- net T8: now also U11.25 (A8)
- net T9: now also U11.24 (A9)
- net MUX: now reaches U1.3 (Q14)
- net MUX: now also U13.4 (C)
- net at U11.11 (D0): now also U12.11 (a)
- net at U11.12 (D1): now also U12.7 (b)
- net at U11.13 (D2): now also U12.4 (c)
- net at U11.15 (D3): now also U12.2 (d)
- net at U11.16 (D4): now also U12.1 (e)
- net at U11.17 (D5): now also U12.10 (f)
- net at U11.18 (D6): now also U12.5 (g)
- net at U11.19 (D7): now also U12.3 (DPX)
- new net: U13.12 (C), U13.6 (Q)
- new net: U13.7 (~{Q}), U14.2 (A0)
- new net: U13.9 (~{Q}), U14.3 (A1)
- new net: U12.6 (CC4), U14.4 (O0)
- new net: U12.8 (CC3), U14.5 (O1)
- new net: U12.9 (CC2), U14.6 (O2)
- new net: U12.12 (CC1), U14.7 (O3)
Other:
- note added: "Display"
- note added: "Minutes Counter"
- note added: "Oscillator"
- note added: "Seconds Counter"
- moved on the sheet: R1, R10, R11, R12, R13, R2, R3, R4, R5, R6, R7, R8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

Commit message: made schematic tweaks, changed README
Parts:
- added C1, C10, C11, C12, C2, C3, C4, C5, C6, C7, C8, C9: 100nF, symbol Device:C
- added D1: LED, symbol Device:LED
- added R14, R15, R16, R17, R18: 2K, symbol Device:R
- added SW2: SW_Push, symbol Switch:SW_Push
- R1: value 330k -> 1M
- R10, R11, R12, R13, R2, R3, R4, R5, R6, R7, R8, R9: value 470 -> 10K
Connections:
- net +5V: now also C1.1, C10.1, C11.1, C12.1, C2.1, C3.1, C4.1, C5.1, C6.1, C7.1, C8.1, C9.1, SW2.1; no longer SW1.12
- net GND: now also C1.2, C10.2, C11.2, C12.2, C2.2, C3.2, C4.2, C5.2, C6.2, C7.2, C8.2, C9.2, D1.1 (K); no longer R10.2, R11.2, R12.2, R2.2, R3.2, R4.2, R5.2, R6.2, R7.2, R8.2, R9.2
- net LOAD: now also SW2.2; no longer SW1.13
- net at U13.7 (~{Q}), U14.2 (A0): now also U11.23 (A11)
- net at U13.9 (~{Q}), U14.3 (A1): now also U11.2 (A12)
- net at U14.4 (O0): now also R14.2; no longer U12.6 (CC4)
- net at U14.5 (O1): now also R15.2; no longer U12.8 (CC3)
- net at U14.6 (O2): now also R16.2; no longer U12.9 (CC2)
- net at U14.7 (O3): now also R17.2; no longer U12.12 (CC1)
- net at U11.19 (D7): now also R18.1; no longer U12.3 (DPX)
- new net: D1.2 (A), R18.2
- new net: R10.2, R11.2, R12.2, R2.2, R3.2, R4.2, R5.2, R6.2, R7.2, R8.2, R9.2
- new net: R14.1, U12.6 (CC4)
- new net: R15.1, U12.8 (CC3)
- new net: R17.1, U12.12 (CC1)
- new net: R16.1, U12.9 (CC2)
Other:
- note added: "Bypass Capacitors"
- moved on the sheet: R1, R13, Y1

Commit message: added screenshots and updated readme
Parts:
- R14, R15, R16, R17: value 2K -> 150
Connections:
- net GND: no longer U2.10 (R_{EXT}), U2.9 (C_{EXT})
Changed lines of the file:
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@@
   (junction (at 267.335 142.24) (diameter 0) (color 0 0 0 0)
   )
-  (junction (at 114.935 66.04) (diameter 0) (color 0 0 0 0)
-  )
   (junction (at 168.275 258.445) (diameter 0) (color 0 0 0 0)
   )
@@
   )
   (wire (pts (xy 269.875 60.96) (xy 269.875 63.5))
-    (stroke (width 0) (type default))
-  )
-  (wire (pts (xy 114.935 66.04) (xy 114.935 71.12))
     (stroke (width 0) (type default))
   )
@@
     )
   )
-  (symbol (lib_id "power:GND") (at 114.935 66.04 270) (unit 1)
-    (in_bom yes) (on_board yes) (dnp no)
-    (property "Reference" "#PWR044" (at 108.585 66.04 0)
-      (effects (font (size 1.27 1.27)) hide)
-    )
-    (property "Value" "GND" (at 111.125 66.04 0)
-      (effects (font (size 1.27 1.27)))
-    )
-    (property "Footprint" "" (at 114.935 66.04 0)
-      (effects (font (size 1.27 1.27)) hide)
-    )
-    (property "Datasheet" "" (at 114.935 66.04 0)
-      (effects (font (size 1.27 1.27)) hide)
-    )
-    (pin "1")
-    (instances
-      (project "clock"
-        (path "/8c136d39-a8f6-46a9-ab02-e0aa4c7091e3"
-          (reference "#PWR044") (unit 1)
-        )
-      )
-    )
-  )
   (symbol (lib_id "My_Symbols:74HC163") (at 165.735 201.93 0) (unit 1)
     (in_bom yes) (on_board yes) (dnp no) (fields_autoplaced)
@@
       (effects (font (size 1.27 1.27)) (justify left))
     )
-    (property "Value" "2K" (at 365.76 213.36 0)
+    (property "Value" "150" (at 365.76 213.36 0)
       (effects (font (size 1.27 1.27)) (justify left))
     )
@@
       (effects (font (size 1.27 1.27)) (justify left))
     )
-    (property "Value" "2K" (at 373.38 213.36 0)
+    (property "Value" "150" (at 373.38 213.36 0)
       (effects (font (size 1.27 1.27)) (justify left))
     )
@@
       (effects (font (size 1.27 1.27)) (justify left))
     )
-    (property "Value" "2K" (at 388.62 213.36 0)
+    (property "Value" "150" (at 388.62 213.36 0)
       (effects (font (size 1.27 1.27)) (justify left))
     )
@@
       (effects (font (size 1.27 1.27)) (justify left))
     )
-    (property "Value" "2K" (at 381 213.36 0)
+    (property "Value" "150" (at 381 213.36 0)
       (effects (font (size 1.27 1.27)) (justify left))
     )
@@
   )
   (symbol (lib_id "My_Symbols:4060") (at 95.25 80.01 0) (unit 1)
-    (in_bom yes) (on_board yes) (dnp no) (fields_autoplaced)
+    (in_bom yes) (on_board yes) (dnp no)
     (property "Reference" "U1" (at 97.4441 58.42 0)
       (effects (font (size 1.27 1.27)) (justify left))
